Commit message: made path accessible outside solver script, added floor and ceiling to base urdf

File: global/drone_RRT_demo/assets/hallway_env1.urdf (robot description, URDF)
Before this commit: robot hallway_env, 5 links, 4 joints
Links:
- added link ceiling; collision box size=10 2.2 0.1; visual box size=10 2.2 0.1
- added link floor; collision box size=10 2.2 0.1; visual box size=10 2.2 0.1
Joints:
- added joint ceiling_joint: type fixed, parent world, child ceiling, origin xyz=0 0 2.05 rpy=0 0 0
- added joint floor_joint: type fixed, parent world, child floor, origin xyz=0 0 -0.05 rpy=0 0 0
